File: SPBT3.0DP2.kicad_pcb (KiCad board)
At the start: 2 copper layers, 27.9 x 25.4 mm, 3 parts, among them CN1 CONN_01X09, CN2 CONN_01X09, U1 SPBT3.0DP2

Commit message: Fix mask clearance.  Set to 0.
Other:
- rule pad_to_mask_clearance: 0.2 -> 0
Changed lines of the file:
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@@
     (pad_size 1.524 1.524)
     (pad_drill 0.762)
-    (pad_to_mask_clearance 0.2)
+    (pad_to_mask_clearance 0)
     (aux_axis_origin 0 0)
     (visible_elements FFFFFF7F)
     (pcbplotparams
-      (layerselection 0x00030_80000001)
+      (layerselection 0x010f8_80000001)
       (usegerberextensions false)
       (excludeedgelayer true)
@@
       (outputformat 1)
       (mirror false)
-      (drillshape 1)
+      (drillshape 0)
       (scaleselection 1)
-      (outputdirectory ""))
+      (outputdirectory Gerbers))
   )
   (net 0 "")
